File: badge-dc24/badge-dc24-with-lcd.kicad_pcb (KiCad board)
At the start: 2 copper layers, 27 parts, among them U1 ESP-12E, U2 TSOP38238, U3 74HC595

Commit message: New design based on learnings from first design
Parts:
- moved Power2 3.31 mm to (123.7, 66.7), turned to 270 degrees
Changed lines of the file:
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@@
   )
   (module Pin_Headers:Pin_Header_Straight_1x02 (layer F.Cu)
-    (at 121.4501 69.1642 180)
+    (at 123.6853 66.7258 270)
     (descr "Through hole pin header")
     (tags "pin header")
-    (fp_text reference Power2 (at 0 -5.1 180) (layer F.SilkS)
-      (effects (font (size 1 1) (thickness 0.15)))
-    )
-    (fp_text value CONN_01X02 (at 0 -3.1 180) (layer F.Fab)
+    (fp_text reference Power2 (at 0 -5.1 270) (layer F.SilkS)
+      (effects (font (size 1 1) (thickness 0.15)))
+    )
+    (fp_text value CONN_01X02 (at 0 -3.1 270) (layer F.Fab)
       (effects (font (size 1 1) (thickness 0.15)))
     )
@@
     (fp_line (start -1.27 1.27) (end -1.27 3.81) (layer F.SilkS) (width 0.15))
     (fp_line (start -1.27 3.81) (end 1.27 3.81) (layer F.SilkS) (width 0.15))
-    (pad 1 thru_hole rect (at 0 0 180) (size 2.032 2.032) (drill 1.016) (layers *.Cu *.Mask F.SilkS)
+    (pad 1 thru_hole rect (at 0 0 270) (size 2.032 2.032) (drill 1.016) (layers *.Cu *.Mask F.SilkS)
       (net 1 +3V3))
-    (pad 2 thru_hole oval (at 0 2.54 180) (size 2.032 2.032) (drill 1.016) (layers *.Cu *.Mask F.SilkS)
+    (pad 2 thru_hole oval (at 0 2.54 270) (size 2.032 2.032) (drill 1.016) (layers *.Cu *.Mask F.SilkS)
       (net 15 GND))
     (model Pin_Headers.3dshapes/Pin_Header_Straight_1x02.wrl
@@
   (segment (start 71.0184 97.0534) (end 71.0184 97.6003) (width 0.5) (layer F.Cu) (net 13))
   (segment (start 71.0184 97.6003) (end 74.2434 100.8253) (width 0.5) (layer F.Cu) (net 13) (status 20))
-  (segment (start 117.555 66.675) (end 117.555 69.2134) (width 0.75) (layer F.Cu) (net 15) (status C00000))
-  (segment (start 117.555 69.2134) (end 117.5566 69.215) (width 0.75) (layer F.Cu) (net 15) (status C00000))
+  (segment (start 117.555 66.675) (end 117.555 69.2134) (width 0.75) (layer F.Cu) (net 15))
+  (segment (start 117.555 69.2134) (end 117.5566 69.215) (width 0.75) (layer F.Cu) (net 15))
   (segment (start 117.555 66.675) (end 121.3993 66.675) (width 0.75) (layer F.Cu) (net 15))
   (segment (start 121.3993 66.675) (end 121.4501 66.6242) (width 0.75) (layer F.Cu) (net 15))

Commit message: Added previous git ref to front copper
Other:
- board text added: "0837d66a419713f16653a0c54959c6bfddd47511"
Changed lines of the file:
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@@
     (area 49.57 58.46 152.36 130.77)
     (thickness 1.6)
-    (drawings 7)
+    (drawings 8)
     (tracks 172)
     (zones 0)
@@
     )
   )
+  (gr_text 0837d66a419713f16653a0c54959c6bfddd47511 (at 96.0882 122.7074) (layer F.Cu)
+    (effects (font (size 1.5 1.5) (thickness 0.3)))
+  )
   (gr_text @elasticninja (at 131.7879 118.5672 45) (layer F.Cu)

Commit message: Added board rev
Other:
- board text added: "v0.2"
Changed lines of the file:
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@@
     (area 49.57 58.46 152.36 130.77)
     (thickness 1.6)
-    (drawings 8)
+    (drawings 10)
     (tracks 172)
     (zones 0)
@@
     )
   )
+  (gr_text v0.2 (at 142.5829 107.6579 45) (layer B.Cu)
+    (effects (font (size 1.5 1.5) (thickness 0.3)) (justify mirror))
+  )
+  (gr_text v0.2 (at 143.0909 107.4801 45) (layer F.Cu)
+    (effects (font (size 1.5 1.5) (thickness 0.3)))
+  )
   (gr_text 0837d66a419713f16653a0c54959c6bfddd47511 (at 96.0882 122.7074) (layer F.Cu)
