File: badge-dc24/badge-dc24-with-lcd-all-smd.kicad_pcb (KiCad board)
At the start: 2 copper layers, 31 parts, among them P1 USB_OTG, U1 ESP-12E, U2 TSOP38238, U3 74HC595, U4 MC78L05ACH

Commit message: Updated git ref
Other:
- board text added: "ed8730e330b6cb4bf74c563c67ffd9e84d4573bc"
- board text removed: "4949bd5106ba81babebe5f0a4540db1eed7f4169"
Changed lines of the file:
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@@
     (effects (font (size 1.5 1.5) (thickness 0.3)))
   )
-  (gr_text 4949bd5106ba81babebe5f0a4540db1eed7f4169 (at 96.1644 123.4948) (layer F.Cu)
+  (gr_text ed8730e330b6cb4bf74c563c67ffd9e84d4573bc (at 96.1644 123.4948) (layer F.Cu)
     (effects (font (size 1.5 1.5) (thickness 0.3)))
   )

Commit message: Cleanup
Parts:
- moved Power1 52.4 mm to (100.8, 67.0)
- moved R1 52.4 mm to (106.1, 67.0)
- moved R10 14.9 mm to (56.8, 94.9)
- moved L4 10.4 mm to (61.7, 104.6)
- moved R4 10.4 mm to (61.8, 110.0)
- moved L1 7.42 mm to (70.7, 104.6)
- moved R7 7.40 mm to (70.6, 110.0)
- moved C3 6.23 mm to (114.8, 69.1), turned to 90 degrees
- moved Power2 4.75 mm to (137.0, 70.4), turned to 180 degrees
- moved L3 4.69 mm to (64.5, 104.6)
- moved R5 4.69 mm to (64.5, 110.0)
- moved C1 4.32 mm to (118.6, 69.1), turned to 90 degrees
- moved U4 3.28 mm to (125.8, 67.9)
- moved C2 2.80 mm to (132.0, 69.1), turned to 90 degrees
- moved L5 1.69 mm to (73.6, 104.6)
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Routing:
- net GND: track 89.4 -> 68.6 mm
- net Net-(D1-Pad1): track 18.4 -> 3.53 mm
- net Net-(C2-Pad1): track 33.1 -> 19.5 mm
- net Net-(L4-Pad1): track 13.7 -> 6.03 mm
- net Net-(L3-Pad1): track 16.6 -> 10.9 mm
- net Net-(L2-Pad1): track 18.6 -> 13.8 mm
- net +3V3: track 10.1 -> 14.8 mm
- net Net-(R9-Pad1): track 15.0 -> 12.3 mm
- net Net-(L5-Pad1): track 12.7 -> 11.4 mm

Commit message: Updated git ref
Other:
- board text added: "062741e576cdccf989905e4a6e1cac9879bf1637"
- board text removed: "ed8730e330b6cb4bf74c563c67ffd9e84d4573bc"
Changed lines of the file:
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@@
     (effects (font (size 1.5 1.5) (thickness 0.3)))
   )
-  (gr_text ed8730e330b6cb4bf74c563c67ffd9e84d4573bc (at 96.1644 123.4948) (layer F.Cu)
+  (gr_text 062741e576cdccf989905e4a6e1cac9879bf1637 (at 96.1644 123.4948) (layer F.Cu)
     (effects (font (size 1.5 1.5) (thickness 0.3)))
   )
