File: badge-dc24/badge-bsides-v0.8.kicad_pcb (KiCad board)
At the start: 2 copper layers, 70 parts, among them P1 USB_OTG, P2 CONN_01X04, U1 ESP-12E, U2 TSOP38238, U3 74HC595, U4 MC78L05ACH, U5 74LS165, U6 CH340H/T, U7 MCP73831, U8 MMA8452QT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

Commit message: Updated git ref on PCB
Other:
- board text added: "ca25f5d94a6718e11e59b6090a1fd236bca68872"
- board text removed: "cc153ddb8d4731039d670fcff0577315d3bf313e"
Changed lines of the file:
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@@
   (page A4)
   (layers
-    (0 F.Cu signal hide)
+    (0 F.Cu signal)
     (31 B.Cu signal)
-    (32 B.Adhes user hide)
+    (32 B.Adhes user)
     (33 F.Adhes user)
-    (34 B.Paste user hide)
+    (34 B.Paste user)
     (35 F.Paste user)
-    (36 B.SilkS user hide)
+    (36 B.SilkS user)
     (37 F.SilkS user)
-    (38 B.Mask user hide)
+    (38 B.Mask user)
     (39 F.Mask user)
     (40 Dwgs.User user)
@@
     (44 Edge.Cuts user)
     (45 Margin user)
-    (46 B.CrtYd user hide)
+    (46 B.CrtYd user)
     (47 F.CrtYd user)
-    (48 B.Fab user hide)
+    (48 B.Fab user)
     (49 F.Fab user)
   )
@@
     (pad_to_mask_clearance 0.2)
     (aux_axis_origin 0 0)
-    (visible_elements FFFFBDFF)
+    (visible_elements FFFFFFFF)
     (pcbplotparams
       (layerselection 0x00030_80000001)
@@
     )
   )
-  (gr_text cc153ddb8d4731039d670fcff0577315d3bf313e (at 49.42078 103.43388 90) (layer B.Cu)
+  (gr_text ca25f5d94a6718e11e59b6090a1fd236bca68872 (at 49.42078 103.43388 90) (layer B.Cu)
     (effects (font (size 1.5 1.5) (thickness 0.3)) (justify mirror))
   )
